Commit message: Launch file with Jeep Display

File: src/jeep_description/urdf/jeep.urdf (robot description, URDF)
Before this commit: robot jeep, 9 links, 8 joints
Links:
- link base_link: geometry collision mesh filename=package://jeep_description/meshes/body_collision.stl scale=0.96 0.96 0.96; visual mesh filename=package://jeep_description/meshes/body.dae scale=1 0.96 1
